Commit message: Set paths to relative, to make repo independent from dev pc.

File: arctos_urdf.urdf (robot description, URDF)
Before this commit: robot arctos, 10 links, 9 joints
Links:
- link Gripper_1: geometry collision mesh filename=meshes/Gripper_1.stl scale=0.001 0.001 0.001; visual mesh filename=meshes/Gripper_1.stl scale=0.001 0.001 0.001
- link Left_jaw_1: geometry collision mesh filename=meshes/Left_jaw_1.stl scale=0.001 0.001 0.001; visual mesh filename=meshes/Left_jaw_1.stl scale=0.001 0.001 0.001
- link Link_1_1: geometry collision mesh filename=meshes/Link_1_1.stl scale=0.001 0.001 0.001; visual mesh filename=meshes/Link_1_1.stl scale=0.001 0.001 0.001
- link Link_2_1: geometry collision mesh filename=meshes/Link_2_1.stl scale=0.001 0.001 0.001; visual mesh filename=meshes/Link_2_1.stl scale=0.001 0.001 0.001
- link Link_3_1: geometry collision mesh filename=meshes/Link_3_1.stl scale=0.001 0.001 0.001; visual mesh filename=meshes/Link_3_1.stl scale=0.001 0.001 0.001
- link Link_4_1: geometry collision mesh filename=meshes/Link_4_1.stl scale=0.001 0.001 0.001; visual mesh filename=meshes/Link_4_1.stl scale=0.001 0.001 0.001
- link Link_5_1: geometry collision mesh filename=meshes/Link_5_1.stl scale=0.001 0.001 0.001; visual mesh filename=meshes/Link_5_1.stl scale=0.001 0.001 0.001
- link Link_6_1: geometry collision mesh filename=meshes/Link_6_1.stl scale=0.001 0.001 0.001; visual mesh filename=meshes/Link_6_1.stl scale=0.001 0.001 0.001
- link Right_jaw_1: geometry collision mesh filename=meshes/Right_jaw_1.stl scale=0.001 0.001 0.001; visual mesh filename=meshes/Right_jaw_1.stl scale=0.001 0.001 0.001
- link base_link: geometry collision mesh filename=meshes/base_link.stl scale=0.001 0.001 0.001; visual mesh filename=meshes/base_link.stl scale=0.001 0.001 0.001

Commit message: Added reading and display of live encoder values.

File: arctos_urdf.urdf (robot description, URDF)
Before this commit: robot arctos, 10 links, 9 joints
Joints:
- joint joint1: limit lower=-3 upper=3 effort=100 velocity=1.0 -> lower=-2.94 upper=2.94 effort=100 velocity=1.0
- joint joint2: limit lower=-1.57 upper=1.57 effort=100 velocity=1.0 -> lower=-0.889 upper=1.91 effort=100 velocity=1.0
- joint joint3: limit lower=-1.57 upper=1.57 effort=100 velocity=1.0 -> lower=-0.6281600193698771 upper=1.45 effort=100 velocity=1.0
- joint joint4: limit lower=-1.57 upper=1.57 effort=100 velocity=1.0 -> lower=-2.94 upper=2.94 effort=100 velocity=1.0
- joint joint5: limit lower=-1.57 upper=1.57 effort=100 velocity=1.0 -> lower=-2.5 upper=2.5 effort=100 velocity=1.0
- joint joint6: limit lower=-1.57 upper=1.57 effort=100 velocity=1.0 -> lower=-2.94 upper=2.94 effort=100 velocity=1.0
